Commit message: fix: adjust robot sensor positions

File: src/lunohod-1/description/camera.xacro (robot description, xacro)
@@ -4,5 +4,5 @@
         <parent link="chassis"/>
         <child link="camera_link"/>
-        <origin xyz="0.276 0 0.181" rpy="0 0 0"/>
+        <origin xyz="0.380 0 0.181" rpy="0 0 0"/>
     </joint>
     <link name="camera_link">

File: src/lunohod-1/description/lidar.xacro (robot description, xacro)
@@ -4,5 +4,5 @@
         <parent link="chassis"/>
         <child link="laser_frame"/>
-        <origin xyz="0.122 0 0.212" rpy="0 0 ${pi}"/>
+        <origin xyz="0.270 0 0.212" rpy="0 0 ${pi}"/>
     </joint>
     <link name="laser_frame">

File: src/lunohod-1/description/robot_core.xacro (robot description, xacro)
@@ -46,5 +46,5 @@
         <parent link="base_link"/>
         <child link="chassis"/>
-        <origin xyz="${-wheel_offset_x} 0 ${-wheel_offset_z}" rpy="0 0 ${pi}"/>
+        <origin xyz="${-wheel_offset_x} 0 ${-wheel_offset_z}" rpy="0 0 0"/>
     </joint>
     <link name="chassis">

Commit message: feat: add velocity limits and adjust camera position for improved navigation

File: src/lunohod-1/description/camera.xacro (robot description, xacro)
@@ -4,5 +4,5 @@
         <parent link="chassis"/>
         <child link="camera_link"/>
-        <origin xyz="0.380 0 0.181" rpy="0 0 0"/>
+        <origin xyz="0.415 0 0.181" rpy="0 0 0"/>
     </joint>
     <link name="camera_link">
